Commit message: updated content

File: body.urdf (robot description, URDF)
Before this commit: robot robot, 9 links, 8 joints
Joints:
- joint BackLeg_LowerBack: axis 1 0 0 -> 0 1 1
- joint FrontLeg_LowerFront: axis 1 0 0 -> 0 1 1
- joint LeftLeg_LowerLeft: axis 0 1 0 -> 0 1 1
- joint RightLeg_LowerRight: axis 0 1 0 -> 0 1 1
- joint Torso_BackLeg: axis 1 0 0 -> 0 1 1
- joint Torso_FrontLeg: axis 1 0 0 -> 0 1 1
- joint Torso_LeftLeg: axis 0 1 0 -> 0 1 1
- joint Torso_RightLeg: axis 0 1 0 -> 0 1 1

Commit message: completed legs up

File: body.urdf (robot description, URDF)
Before this commit: robot robot, 9 links, 8 joints
Joints:
- joint BackLeg_LowerBack: axis 0 1 1 -> 0 -1 0
- joint FrontLeg_LowerFront: axis 0 1 1 -> 0 -1 0
- joint LeftLeg_LowerLeft: axis 0 1 1 -> 0 -1 0
- joint RightLeg_LowerRight: axis 0 1 1 -> 0 -1 0
- joint Torso_BackLeg: axis 0 1 1 -> 0 1 0
- joint Torso_FrontLeg: axis 0 1 1 -> 0 1 0
- joint Torso_LeftLeg: axis 0 1 1 -> 0 1 0
- joint Torso_RightLeg: axis 0 1 1 -> 0 1 0

Commit message: finished legsup

File: body.urdf (robot description, URDF)
Before this commit: robot robot, 9 links, 8 joints
Joints:
- joint BackLeg_LowerBack: axis 0 -1 0 -> 0 1 0
- joint FrontLeg_LowerFront: axis 0 -1 0 -> 0 1 0
- joint LeftLeg_LowerLeft: axis 0 -1 0 -> 0 1 0
- joint RightLeg_LowerRight: axis 0 -1 0 -> 0 1 0

Commit message: Finished deliverable 3

File: body.urdf (robot description, URDF)
Before this commit: robot robot, 9 links, 8 joints
Links:
- link BackLeg: geometry collision box size=0.2 1.3729335165261551 0.2; visual box size=0.2 1.3729335165261551 0.2
- link FrontLeg: geometry collision box size=0.2 2.4105288999540995 0.2; visual box size=0.2 2.4105288999540995 0.2
- link LeftLeg: geometry collision box size=1.126220416926897 0.2 0.2; visual box size=1.126220416926897 0.2 0.2
- link LowerBack: geometry collision box size=0.2 0.2 1.0148282919145082; visual box size=0.2 0.2 1.0148282919145082
- link LowerFront: geometry collision box size=0.2 0.2 0.8909737456892562; visual box size=0.2 0.2 0.8909737456892562
- link LowerLeft: geometry collision box size=0.2 0.2 2.229926729572571; visual box size=0.2 0.2 2.229926729572571
- link LowerRight: geometry collision box size=0.2 0.2 1.431729674563428; visual box size=0.2 0.2 1.431729674563428
- link RightLeg: geometry collision box size=0.842126838513556 0.2 0.2; visual box size=0.842126838513556 0.2 0.2
Joints:
- joint BackLeg_LowerBack: axis 0 1 1 -> 0 1 0; origin xyz=0 -1 0 rpy=0 0 0 -> xyz=0 -1.3729335165261551 0 rpy=0 0 0
- joint FrontLeg_LowerFront: axis 0 1 1 -> 0 1 0; origin xyz=0 1 0 rpy=0 0 0 -> xyz=0 2.4105288999540995 0 rpy=0 0 0
- joint LeftLeg_LowerLeft: axis 0 1 1 -> 0 1 0; origin xyz=-1 0 0 rpy=0 0 0 -> xyz=-1.126220416926897 0 0 rpy=0 0 0
- joint RightLeg_LowerRight: axis 0 1 1 -> 0 1 0; origin xyz=1 0 0 rpy=0 0 0 -> xyz=0.842126838513556 0 0 rpy=0 0 0
- joint Torso_BackLeg: axis 0 1 1 -> 0 1 0; origin xyz=0 -0.5 1 rpy=0 0 0 -> xyz=0 -0.5 3 rpy=0 0 0
- joint Torso_FrontLeg: axis 0 1 1 -> 0 1 0; origin xyz=0 0.5 1 rpy=0 0 0 -> xyz=0 0.5 3 rpy=0 0 0
- joint Torso_LeftLeg: axis 0 1 1 -> 0 1 0; origin xyz=-0.5 0 1 rpy=0 0 0 -> xyz=-0.5 0 3 rpy=0 0 0
- joint Torso_RightLeg: axis 0 1 1 -> 0 1 0; origin xyz=0.5 0 1 rpy=0 0 0 -> xyz=0.5 0 3 rpy=0 0 0

Commit message: Completed mind and body test

File: body.urdf (robot description, URDF)
Before this commit: robot robot, 9 links, 8 joints
Links:
- link BackLeg: geometry collision box size=0.2 0.943763667765952 0.2; visual box size=0.2 0.943763667765952 0.2
- link FrontLeg: geometry collision box size=0.2 1.376634569382718 0.2; visual box size=0.2 1.376634569382718 0.2
- link LeftLeg: geometry collision box size=1.301267934162524 0.2 0.2; visual box size=1.301267934162524 0.2 0.2
- link LowerBack: geometry collision box size=0.2 0.2 0.6462354553456419; visual box size=0.2 0.2 0.6462354553456419
- link LowerFront: geometry collision box size=0.2 0.2 1.0271371248677397; visual box size=0.2 0.2 1.0271371248677397
- link LowerLeft: geometry collision box size=0.2 0.2 1.041233371922241; visual box size=0.2 0.2 1.041233371922241
- link LowerRight: geometry collision box size=0.2 0.2 0.8710460859184639; visual box size=0.2 0.2 0.8710460859184639
- link RightLeg: geometry collision box size=0.8806500102345981 0.2 0.2; visual box size=0.8806500102345981 0.2 0.2
Joints:
- joint BackLeg_LowerBack: origin xyz=0 -1.3729335165261551 0 rpy=0 0 0 -> xyz=0 -0.943763667765952 0 rpy=0 0 0
- joint FrontLeg_LowerFront: origin xyz=0 2.4105288999540995 0 rpy=0 0 0 -> xyz=0 1.376634569382718 0 rpy=0 0 0
- joint LeftLeg_LowerLeft: origin xyz=-1.126220416926897 0 0 rpy=0 0 0 -> xyz=-1.301267934162524 0 0 rpy=0 0 0
- joint RightLeg_LowerRight: origin xyz=0.842126838513556 0 0 rpy=0 0 0 -> xyz=0.8806500102345981 0 0 rpy=0 0 0

Commit message: completed reg leg simulations

File: body.urdf (robot description, URDF)
Before this commit: robot robot, 9 links, 8 joints
Joints:
- joint BackLeg_LowerBack: axis 0 1 1 -> 0 1 0
- joint FrontLeg_LowerFront: axis 0 1 1 -> 0 1 0
- joint LeftLeg_LowerLeft: axis 0 1 1 -> 0 1 0
- joint RightLeg_LowerRight: axis 0 1 1 -> 0 1 0
- joint Torso_BackLeg: axis 0 1 1 -> 0 1 0
- joint Torso_FrontLeg: axis 0 1 1 -> 0 1 0
- joint Torso_LeftLeg: axis 0 1 1 -> 0 1 0
- joint Torso_RightLeg: axis 0 1 1 -> 0 1 0
